Commit message: added lidar support

File: src/terratrek_robot/description/robot.urdf.xacro (robot description, xacro)
@@ -2,4 +2,5 @@
 <robot xmlns:xacro="http://www.ros.org/wiki/xacro"  name="robot">
     <xacro:include filename="robot_core.xacro" />
+    <xacro:include filename="lidar.xacro"/>
     <xacro:include filename="ros2_control.xacro" />
     <!--xacro:include filename="gazebo_control.xacro"/-->

File: src/terratrek_robot/description/robot_core.xacro (robot description, xacro)
@@ -60,6 +60,6 @@
         <origin xyz="0 -${arm_offset} -0.038"/>
         <axis xyz="0 1 0"/>
-        <limit effort="100" velocity="2.0" lower="-${pi/6}" upper="${pi/6}" />
-        <dynamics damping="3" friction="0.025"/>
+        <limit effort="100" velocity="5.0" lower="-${pi/6}" upper="${pi/6}" />
+        <dynamics damping="10" friction="0.25"/>
     </joint>
     <link name="right_arm_inner">
@@ -87,7 +87,7 @@
         <origin xyz="0 ${arm_offset} -0.038"/>
         <axis xyz="0 1 0"/>
-        <limit effort="100" velocity="2.0" lower="-${pi/6}" upper="${pi/6}"/>
+        <limit effort="100" velocity="5.0" lower="-${pi/6}" upper="${pi/6}"/>
         <mimic joint="right_arm_inner_joint" multiplier="1.0"/>
-        <dynamics damping="3" friction=".025"/>
+        <dynamics damping="10" friction="0.25"/>
     </joint>
     <link name="left_arm_inner">
@@ -110,11 +110,11 @@
     </link>
     <!-- OUTER RIGHT ARM-->
-    <joint name="right_arm_outer_joint" type="prismatic">
+    <joint name="right_arm_outer_joint" type="fixed">
         <parent link="right_arm_inner"/>
         <child link="right_arm_outer"/>
         <origin xyz="${arm_outer_offset} -${arm_width + .001} 0"/>
         <axis xyz="1 0 0"/>
-        <limit effort="2" velocity="0.01" upper="0.2"/>
-        <dynamics damping="3" friction="0.025"/>
+        <!--limit effort="100" velocity="0.01" upper="0.2"/-->
+        <!--dynamics damping="3" friction="0.025"/-->
     </joint>
     <link name="right_arm_outer">
@@ -137,11 +137,11 @@
     </link>
     <!-- OUTER LEFT ARM-->
-    <joint name="left_arm_outer_joint" type="prismatic">
+    <joint name="left_arm_outer_joint" type="fixed">
         <parent link="left_arm_inner"/>
         <child link="left_arm_outer"/>
         <origin xyz="${arm_outer_offset} ${arm_width + .001} 0"/>
         <axis xyz="1 0 0"/>
-        <limit effort="2" velocity="0.01" upper=".2"/>
-        <dynamics damping="3" friction="0.025"/>
+        <!--limit effort="100" velocity="0.01" upper=".2"/-->
+        <!--dynamics damping="3" friction="0.025"/-->
     </joint>
     <link name="left_arm_outer">
@@ -371,4 +371,6 @@
     <gazebo reference="FR_wheel">
         <material>Gazebo/Black</material>
+        <mu1 value="0.001"/>
+        <!--mu2 value="0.001"/-->
     </gazebo>
     <gazebo reference="BR_wheel">
@@ -377,4 +379,6 @@
     <gazebo reference="FL_wheel">
         <material>Gazebo/Black</material>
+        <mu1 value="0.001"/>
+        <!--mu2 value="0.001"/-->
     </gazebo>
     <gazebo reference="BL_wheel">
