Commit message: slam added params need tuning

File: src/terratrek_robot/description/robot_core.xacro (robot description, xacro)
@@ -18,4 +18,5 @@
    <xacro:property name="wheel_offset_y" value="0.2667"/>
    <xacro:property name="wheel_offset_x" value="0.27305"/>
+   <xacro:property name="rotation_limit" value="${0/6}"/>
     <material name="white">
         <color rgba="1 1 1 1" />
@@ -30,4 +31,12 @@
     <link name="base_link">
     </link>
+    <!-- BASE FOOTPRINT-->
+    <joint name="base_footprint_joint" type="fixed">
+        <parent link="base_link"/>
+        <child link="base_footprint"/>
+        <origin xyz="0 0 0" rpy="0 0 0"/>
+    </joint>
+    <link name="base_footprint">
+    </link>
     <!-- CHASSIS LINK -->
     <joint name="chassis_joint" type="fixed">
@@ -60,5 +69,5 @@
         <origin xyz="0 -${arm_offset} -0.038"/>
         <axis xyz="0 1 0"/>
-        <limit effort="100" velocity="5.0" lower="-${pi/6}" upper="${pi/6}" />
+        <limit effort="100" velocity="5.0" lower="-${rotation_limit}" upper="${rotation_limit}" />
         <dynamics damping="10" friction="0.25"/>
     </joint>
@@ -87,5 +96,5 @@
         <origin xyz="0 ${arm_offset} -0.038"/>
         <axis xyz="0 1 0"/>
-        <limit effort="100" velocity="5.0" lower="-${pi/6}" upper="${pi/6}"/>
+        <limit effort="100" velocity="5.0" lower="-${rotation_limit}" upper="${rotation_limit}"/>
         <mimic joint="right_arm_inner_joint" multiplier="1.0"/>
         <dynamics damping="10" friction="0.25"/>

File: src/terratrek_robot/description/ros2_control.xacro (robot description, xacro)
@@ -7,6 +7,6 @@
         <joint name="FL_wheel_joint">
             <command_interface name= "velocity">
-                <param name="min">-10</param>
-                <param name="max">20</param>
+                <param name="min">-2.5</param>
+                <param name="max">2.5</param>
             </command_interface>
             <state_interface name= "velocity"/>
@@ -15,6 +15,6 @@
         <joint name="FR_wheel_joint">
             <command_interface name= "velocity">
-                <param name="min">-10</param>
-                <param name="max">20</param>
+                <param name="min">-2.5</param>
+                <param name="max">2.5</param>
             </command_interface>
             <state_interface name= "velocity"/>
@@ -23,6 +23,6 @@
         <joint name="BL_wheel_joint">
             <command_interface name= "velocity">
-                <param name="min">-10</param>
-                <param name="max">20</param>
+                <param name="min">-2.5</param>
+                <param name="max">2.5</param>
             </command_interface>
             <state_interface name= "velocity"/>
@@ -31,6 +31,6 @@
         <joint name="BR_wheel_joint">
             <command_interface name= "velocity">
-                <param name="min">-10</param>
-                <param name="max">20</param>
+                <param name="min">-2.5</param>
+                <param name="max">2.5</param>
             </command_interface>
             <state_interface name= "velocity"/>
@@ -39,6 +39,6 @@
         <!--joint name="right_arm_inner_joint">
             <command_interface name="position">
-            <param name="min">-0.125</param>
-            <param name="max">.125</param>
+            <param name="min">-0.122.5</param>
+            <param name="max">.122.5</param>
             </command_interface>
             <state_interface name="position"/>
@@ -47,5 +47,5 @@
             <command_interface name="position">
             <param name="min">0</param>
-            <param name="max">100</param>
+            <param name="max">2.50</param>
             </command_interface>
             <state_interface name="position"/>
@@ -54,5 +54,5 @@
             <command_interface name="position">
             <param name="min">0</param>
-            <param name="max">100</param>
+            <param name="max">2.50</param>
             </command_interface>
             <state_interface name="position"/>
