Commit message: Nav2 fully working

File: src/terratrek_robot/description/lidar.xacro (robot description, xacro)
@@ -13,9 +13,9 @@
             <material name="red"/>
         </visual>
-        <collision>
+        <!-- <collision>
             <geometry>
                 <cylinder radius="0.03" length="0.04"/>
             </geometry>
-        </collision>
+        </collision> -->
         <xacro:inertial_cylinder mass="0.1" length="0.04" radius="0.05">
             <origin xyz="0 0 0" rpy="0 0 0"/>

File: src/terratrek_robot/description/robot_core.xacro (robot description, xacro)
@@ -18,5 +18,5 @@
    <xacro:property name="wheel_offset_y" value="0.2667"/>
    <xacro:property name="wheel_offset_x" value="0.27305"/>
-   <xacro:property name="rotation_limit" value="${0/6}"/>
+   <xacro:property name="rotation_limit" value="${pi/6}"/>
     <material name="white">
         <color rgba="1 1 1 1" />
@@ -70,5 +70,5 @@
         <axis xyz="0 1 0"/>
         <limit effort="100" velocity="5.0" lower="-${rotation_limit}" upper="${rotation_limit}" />
-        <dynamics damping="10" friction="0.25"/>
+        <dynamics damping="1" friction="0.25"/>
     </joint>
     <link name="right_arm_inner">
@@ -97,6 +97,5 @@
         <axis xyz="0 1 0"/>
         <limit effort="100" velocity="5.0" lower="-${rotation_limit}" upper="${rotation_limit}"/>
-        <mimic joint="right_arm_inner_joint" multiplier="1.0"/>
-        <dynamics damping="10" friction="0.25"/>
+        <mimic joint="right_arm_inner_joint" multiplier="-1.0"/>
     </joint>
     <link name="left_arm_inner">
@@ -119,11 +118,11 @@
     </link>
     <!-- OUTER RIGHT ARM-->
-    <joint name="right_arm_outer_joint" type="fixed">
+    <joint name="right_arm_outer_joint" type="prismatic">
         <parent link="right_arm_inner"/>
         <child link="right_arm_outer"/>
         <origin xyz="${arm_outer_offset} -${arm_width + .001} 0"/>
         <axis xyz="1 0 0"/>
-        <!--limit effort="100" velocity="0.01" upper="0.2"/-->
-        <!--dynamics damping="3" friction="0.025"/-->
+        <limit effort="100" velocity="0.01" upper="0"/>
+        <dynamics damping="3" friction="0.025"/>
     </joint>
     <link name="right_arm_outer">
@@ -146,11 +145,11 @@
     </link>
     <!-- OUTER LEFT ARM-->
-    <joint name="left_arm_outer_joint" type="fixed">
+    <joint name="left_arm_outer_joint" type="prismatic">
         <parent link="left_arm_inner"/>
         <child link="left_arm_outer"/>
         <origin xyz="${arm_outer_offset} ${arm_width + .001} 0"/>
         <axis xyz="1 0 0"/>
-        <!--limit effort="100" velocity="0.01" upper=".2"/-->
-        <!--dynamics damping="3" friction="0.025"/-->
+        <limit effort="100" velocity="0.01" upper="0"/>
+        <dynamics damping="3" friction="0.025"/>
     </joint>
     <link name="left_arm_outer">
@@ -362,17 +361,17 @@
     <gazebo>
         <plugin name="joint_states" filename="libgazebo_ros_joint_state_publisher.so">
-        <ros>
-            <!-- <namespace>/br</namespace> -->
-            <remapping>~/out:=joint_states</remapping>
-        </ros>
-        <update_rate>30</update_rate>
-        <joint_name>right_arm_inner_joint</joint_name>
-        <joint_name>right_arm_outer_joint</joint_name>
-        <joint_name>left_arm_inner_joint</joint_name>
-        <joint_name>left_arm_outer_joint</joint_name>
-        <joint_name>BL_wheel_joint</joint_name>
-        <joint_name>BR_wheel_joint</joint_name>
-        <joint_name>FL_wheel_joint</joint_name>
-        <joint_name>FR_wheel_joint</joint_name>
+            <ros>
+                <!-- <namespace>/br</namespace> -->
+                <remapping>~/out:=joint_states</remapping>
+            </ros>
+            <update_rate>30</update_rate>
+            <joint_name>right_arm_inner_joint</joint_name>
+            <joint_name>right_arm_outer_joint</joint_name>
+            <joint_name>left_arm_inner_joint</joint_name>
+            <joint_name>left_arm_outer_joint</joint_name>
+            <joint_name>BL_wheel_joint</joint_name>
+            <joint_name>BR_wheel_joint</joint_name>
+            <joint_name>FL_wheel_joint</joint_name>
+            <joint_name>FR_wheel_joint</joint_name>
         </plugin>
     </gazebo>

File: src/terratrek_robot/description/ros2_control.xacro (robot description, xacro)
@@ -44,18 +44,23 @@
             <state_interface name="position"/>
         </joint-->
-        <!--joint name="right_arm_outer_joint">
-            <command_interface name="position">
+        <!-- <joint name="right_arm_outer_joint">
+            <command_interface name="effort">
             <param name="min">0</param>
-            <param name="max">500</param>
+            <param name="max">5</param>
+            </command_interface>
+            <state_interface name="position">
+            <param name="initial_value">0.0</param>
+            </state_interface>
+        </joint> -->
+        <!-- <joint name="left_arm_outer_joint">
+            <command_interface name="effort">
+            <param name="min">0</param>
+            <param name="max">5</param>
             </command_interface>
             <state_interface name="position"/>
-        </joint-->
-        <!--joint name="left_arm_outer_joint">
-            <command_interface name="position">
-            <param name="min">0</param>
-            <param name="max">500</param>
-            </command_interface>
-            <state_interface name="position"/>
-        </joint-->
+            <state_interface name="position">
+            <param name="initial_value">0.0</param>
+            </state_interface>
+        </joint> -->
     </ros2_control>
     <gazebo>
@@ -63,4 +68,11 @@
             <parameters>$(find terratrek_robot)/config/my_controllers.yaml</parameters>
         </plugin>
+        <plugin filename="libroboticsgroup_upatras_gazebo_mimic_joint_plugin.so" name="mimic_robotiq_85_1">
+            <joint>left_arm_inner_joint</joint>
+            <mimicJoint>right_arm_inner_joint</mimicJoint>
+            <multiplier>-1.0</multiplier>
+            <offset>0.0</offset>
+            <maxEffort>5.0</maxEffort>
+        </plugin>
     </gazebo>
 </robot>
