Commit message: start of hardware

File: src/terratrek_robot/description/ros2_control.xacro (robot description, xacro)
@@ -37,30 +37,4 @@
             <state_interface name= "position"/>
         </joint>
-        <!--joint name="right_arm_inner_joint">
-            <command_interface name="position">
-            <param name="min">-0.1250</param>
-            <param name="max">.1250</param>
-            </command_interface>
-            <state_interface name="position"/>
-        </joint-->
-        <!-- <joint name="right_arm_outer_joint">
-            <command_interface name="effort">
-            <param name="min">0</param>
-            <param name="max">5</param>
-            </command_interface>
-            <state_interface name="position">
-            <param name="initial_value">0.0</param>
-            </state_interface>
-        </joint> -->
-        <!-- <joint name="left_arm_outer_joint">
-            <command_interface name="effort">
-            <param name="min">0</param>
-            <param name="max">5</param>
-            </command_interface>
-            <state_interface name="position"/>
-            <state_interface name="position">
-            <param name="initial_value">0.0</param>
-            </state_interface>
-        </joint> -->
     </ros2_control>
     <gazebo>
@@ -76,3 +50,23 @@
         </plugin>
     </gazebo>
+    <transmission name="trans_extender_left">
+        <type>transmission_interface/SimpleTransmission</type>
+            <joint name="left_arm_outer_joint">
+                <hardwareInterface>hardware_interface/EffortJointInterface</hardwareInterface>
+            </joint>
+        <actuator name="motor_extender_left">
+            <hardwareInterface>hardware_interface/EffortJointInterface</hardwareInterface>
+            <mechanicalReduction>1</mechanicalReduction>
+        </actuator>
+    </transmission>
+    <transmission name="trans_extender_right">
+        <type>transmission_interface/SimpleTransmission</type>
+            <joint name="right_arm_outer_joint">
+                <hardwareInterface>hardware_interface/EffortJointInterface</hardwareInterface>
+            </joint>
+        <actuator name="motor_extender_right">
+            <hardwareInterface>hardware_interface/EffortJointInterface</hardwareInterface>
+            <mechanicalReduction>1</mechanicalReduction>
+        </actuator>
+    </transmission>
 </robot>

Commit message: start of day 10 27

File: src/terratrek_robot/description/ros2_control.xacro (robot description, xacro)
@@ -1,41 +1,91 @@
 <?xml version="1.0"?>
 <robot xmlns:xacro="http://www.ros.org/wiki/xacro">
-    <ros2_control name= "GazeboSystem" type= "system">
-        <hardware>
-            <plugin>gazebo_ros2_control/GazeboSystem</plugin>
-        </hardware>
-        <joint name="FL_wheel_joint">
-            <command_interface name= "velocity">
-                <param name="min">-50</param>
-                <param name="max">50</param>
-            </command_interface>
-            <state_interface name= "velocity"/>
-            <state_interface name= "position"/>
-        </joint>
-        <joint name="FR_wheel_joint">
-            <command_interface name= "velocity">
-                <param name="min">-50</param>
-                <param name="max">50</param>
-            </command_interface>
-            <state_interface name= "velocity"/>
-            <state_interface name= "position"/>
-        </joint>
-        <joint name="BL_wheel_joint">
-            <command_interface name= "velocity">
-                <param name="min">-50</param>
-                <param name="max">50</param>
-            </command_interface>
-            <state_interface name= "velocity"/>
-            <state_interface name= "position"/>
-        </joint>
-        <joint name="BR_wheel_joint">
-            <command_interface name= "velocity">
-                <param name="min">-50</param>
-                <param name="max">50</param>
-            </command_interface>
-            <state_interface name= "velocity"/>
-            <state_interface name= "position"/>
-        </joint>
-    </ros2_control>
+    <xacro:unless value="$(arg sim_mode)">
+        <ros2_control name="RealRobot" type="system">
+            <hardware>
+                <plugin>diffdrive_arduino/DiffDriveArduino</plugin>
+                <param name="BL_wheel_name">BL_wheel_joint</param>
+                <param name="BR_wheel_name">BR_wheel_joint</param>
+                <param name="FL_wheel_name">FL_wheel_joint</param>
+                <param name="FR_wheel_name">FR_wheel_joint</param>
+                <param name="loop_rate">30</param>
+                <param name="device">/dev/ttyUSB0</param>
+                <param name="baud_rate">57600</param>
+                <param name="timeou_ms">1000</param>
+                <param name="enc_counts_per_rev">28</param>
+            </hardware>
+            <joint name="BL_wheel_joint">
+                <command_interface name="velocity">
+                    <param name="min">-10</param>
+                    <param name="max">10</param>
+                </command_interface>
+                <state_interface name="velocity"/>
+                <state_interface name="position"/>
+            </joint>
+            <joint name="BR_wheel_joint">
+                <command_interface name="velocity">
+                    <param name="min">-10</param>
+                    <param name="max">10</param>
+                </command_interface>
+                <state_interface name="velocity"/>
+                <state_interface name="position"/>
+            </joint>
+            <joint name="FL_wheel_joint">
+                <command_interface name="velocity">
+                    <param name="min">-10</param>
+                    <param name="max">10</param>
+                </command_interface>
+                <state_interface name="velocity"/>
+                <state_interface name="position"/>
+            </joint>
+            <joint name="FR_wheel_joint">
+                <command_interface name="velocity">
+                    <param name="min">-10</param>
+                    <param name="max">10</param>
+                </command_interface>
+                <state_interface name="velocity"/>
+                <state_interface name="position"/>
+            </joint>
+        </ros2_control>
+    </xacro:unless>
+    <xacro:if value="$(arg sim_mode)">
+        <ros2_control name= "GazeboSystem" type= "system">
+            <hardware>
+                <plugin>gazebo_ros2_control/GazeboSystem</plugin>
+            </hardware>
+            <joint name="FL_wheel_joint">
+                <command_interface name= "velocity">
+                    <param name="min">-50</param>
+                    <param name="max">50</param>
+                </command_interface>
+                <state_interface name= "velocity"/>
+                <state_interface name= "position"/>
+            </joint>
+            <joint name="FR_wheel_joint">
+                <command_interface name= "velocity">
+                    <param name="min">-50</param>
+                    <param name="max">50</param>
+                </command_interface>
+                <state_interface name= "velocity"/>
+                <state_interface name= "position"/>
+            </joint>
+            <joint name="BL_wheel_joint">
+                <command_interface name= "velocity">
+                    <param name="min">-50</param>
+                    <param name="max">50</param>
+                </command_interface>
+                <state_interface name= "velocity"/>
+                <state_interface name= "position"/>
+            </joint>
+            <joint name="BR_wheel_joint">
+                <command_interface name= "velocity">
+                    <param name="min">-50</param>
+                    <param name="max">50</param>
+                </command_interface>
+                <state_interface name= "velocity"/>
+                <state_interface name= "position"/>
+            </joint>
+        </ros2_control>
+    </xacro:if>
     <gazebo>
         <plugin name="skid_steer_drive" filename="libgazebo_ros2_control.so">
@@ -50,23 +100,3 @@
         </plugin>
     </gazebo>
-    <transmission name="trans_extender_left">
-        <type>transmission_interface/SimpleTransmission</type>
-            <joint name="left_arm_outer_joint">
-                <hardwareInterface>hardware_interface/EffortJointInterface</hardwareInterface>
-            </joint>
-        <actuator name="motor_extender_left">
-            <hardwareInterface>hardware_interface/EffortJointInterface</hardwareInterface>
-            <mechanicalReduction>1</mechanicalReduction>
-        </actuator>
-    </transmission>
-    <transmission name="trans_extender_right">
-        <type>transmission_interface/SimpleTransmission</type>
-            <joint name="right_arm_outer_joint">
-                <hardwareInterface>hardware_interface/EffortJointInterface</hardwareInterface>
-            </joint>
-        <actuator name="motor_extender_right">
-            <hardwareInterface>hardware_interface/EffortJointInterface</hardwareInterface>
-            <mechanicalReduction>1</mechanicalReduction>
-        </actuator>
-    </transmission>
 </robot>
